File: pcb/uacs-bottom.sch (EAGLE design)
At the start: 156 parts, among them IC1 TSC2046, IC2 MFRC531, IC3 W5100, IC4 STM809L, P1 MI0283QT-11, Q1 MMBT2222, Q2 13.56MHz, Q3 2N7002, Q4 25MHz, Q5 BSS138, Q6 BSS138, Q7 16MHz, T1 TL2575-05, T2 LM3940IMP-3.3, T3 BC847, U2 ATMEGA640/1280/2560, X1 7499210124A, X3 MICROSD

Commit message: initial commit v2.0
Parts:
- removed B1: CDBHD2100-G, rectifier:B10S
- removed C1, C12, C14, C2, C3, C4, C5, C52, C55, C56, C57, C58, C59, C6, C60, C7: 100n, rcl:C-EUC0603
- removed C10, C11: 15p, rcl:C-EUC0603
- removed C13, C8, C9: 56p, rcl:C-EUC0603
- removed C15, C16: 68p, rcl:C-EUC0603
- removed C17: 1n, rcl:C-EUC0603
- removed C18, C19, C20, C21: 20p, rcl:C-EUC0603
- removed C22, C23: 220p, rcl:C-EUC0603
- removed C24, C25: 200p, rcl:C-EUC0603
- removed C47: 100u, rcl:CPOL-EUG
- removed C48: 470u, rcl:CPOL-EUG
- removed C49: 470n, rcl:CPOL-EUB
- removed C50: 33u, rcl:CPOL-EUD
- removed C51: 33u, rcl:CPOL-EUC/6032-28R
- removed C53, C54: 22p, rcl:C-EUC0603
- removed D1, D2, D5: BAT54, diode:BAT54
- removed D4: PMEG6020ER, adafruit:DIODESOD-123
- removed FTDI: 1X6, pinheader-smd:1X6
- removed IC1: TSC2046, TSC2046:TSC2046
- removed IC2: MFRC531, mfrc531:MFRC531
- removed IC4: STM809L, stm809:STM809
- removed ISP: ISP, pinheader-smd:2X3
- removed L1, L2, L3: 22n, SparkFun-Passives:INDUCTOR0603
- removed L4, L5: 1u, SparkFun-Passives:INDUCTOR0603
- removed L8: SRR1260-331K, EagleLibrary_Wuerth_Elektronik_eiSos_V6_20140807:WE-PD_1260/1245/1280/1210
- removed P1: MI0283QT-11, MI0283QT-11:MI0283QT-11
- removed PWR: GREEN, adafruit:LEDCHIPLED_0603
- removed Q1: MMBT2222, SparkFun-DiscreteSemi:TRANSISTOR_NPNMMBT2222A
- removed Q2: 13.56MHz, adafruit:CRYSTALSM49
- removed Q5, Q6: BSS138, SparkFun-DiscreteSemi:MOSFET-NCHANNELBSS138
- removed Q7: 16MHz, adafruit:CRYSTALSM49
- removed R1, R13, R2, R44, R45: 1k, rcl:R-EU_R0603
- removed R10, R11, R12, R32, R33, R34, R35, R36, R38, R41, R42, R43, R46, R48, R49: 10k, rcl:R-EU_R0603
- removed R14, R15: 0R, rcl:R-EU_R0603
- removed R3, R4: 10K, rcl:R-EU_R0603
- removed R31: 5R6, rcl:R-EU_R0603
- removed R37, R39, R40: 4k7, rcl:R-EU_R0603
- removed R47, R5, R6, R7, R8: 100R, rcl:R-EU_R0603
- removed R9: 820R, rcl:R-EU_R0603
- removed RFID: BLUE, adafruit:LEDCHIPLED_0603
- removed SP1: PS1240P02BT, adafruit:SPEAKER/PS12
- removed T1: TL2575-05, tl2575:TL2575-05
- removed T2: LM3940IMP-3.3, LM3940:LM3940IMP-3.3
- removed T3: BC847, transistor:BC847
- removed TP1, TP2: PTR1B1,27, testpad:PTR1B1,27
- removed U1: (no value), microbuilder:74HC4050DTSSOP
- removed U2: ATMEGA640/1280/2560, SparkFun-DigitalIC:ATMEGA2560AU
- removed X3: MICROSD, adafruit:MICROSD
- removed X5: (no value), con-weidmueller-sl35:180-10
- removed X6: (no value), SparkFun-Connectors:PINHD-2X10
- removed X7: (no value), con-jack:JACK-PLUG1
Connections:
- removed net !PENIRQ: IC1.!PENIRQ, U2.(RXD1/INT2)PD2
- removed net !RESET: D2.C, D5.C, IC4.!RST, U1.4A
- removed net !RESET_PRG: C60.1, D5.A, ISP.5, R49.2, U2.RESET
- removed net !RFID_IRQ: IC2.!IRQ, U2.(OC3B/INT4)PE4
- removed net !RFID_SS: IC2.ALE/AS/NASTREB/NSS, R12.1, U2.PL4(OC5B)
- removed net !SD_SS: R42.1, U1.5A, U2.PL2(T5)
- removed net !SD_SS_3V3: U1.5Y, X3.CS
- removed net !TFT_SS: R41.1, U1.3A, U2.PL6
- removed net !TFT_SS_3V3: P1.CSX, U1.3Y
- removed net !TOUCH_SS: IC1.!CS, R4.1, U2.PL7
- removed net !WIZ_IRQ: R34.2, U2.(TXD1/INT3)PD3
- removed net !WIZ_SS: R43.1, U1.6A, U2.PL3(OC5A)
- removed net A1: U2.(ADC0)PF0, X5.3, X6.15
- removed net A2: U2.(ADC1)PF1, X5.2, X6.16
- removed net A3: U2.(ADC2)PF2, X5.1, X6.17
- removed net A4: U2.(ADC3)PF3, X6.18
- removed net A5: U2.(ADC4/TCK)PF4, X6.19
- removed net A6: U2.(ADC5/TMS)PF5, X6.20
- removed net ANT_RX: C14.1, IC2.RX, R13.1, R9.2
- removed net ANT_TX1: IC2.TX1, L4.1
- removed net ANT_TX2: IC2.TX2, L5.1
- removed net AVDD: C12.1, IC2.AVDD, L3.1
- removed net BUZZ: R45.1, U2.(OC0A/OC1C/PCINT7)PB7
- removed net COIL1: R14.2
- removed net COIL2: R15.2
- removed net D1: U2.(OC0B)PG5, X6.8
- removed net D2: U2.(OC3A/AIN1)PE3, X5.6, X6.9
- removed net D3: U2.(OC3C/INT5)PE5, X6.10
- removed net D4: U2.PH3(OC4A), X5.5, X6.11
- removed net D5: U2.PH4(OC4B), X6.12
- removed net D6: U2.PH5(OC4C), X5.4, X6.13
- removed net D7: U2.PH6(OC2B), X6.14
- removed net DVDD: C7.1, IC2.DVDD, IC2.NRD/NDS/NDSTRB, IC2.NWR/R/NW/NWRITE, L2.1, R10.2, R12.2
- removed net LED_RFID: R47.1, U2.PL1(ICP5)
- removed net MISO: IC1.DOUT, IC2.AD0/D0, R38.2, R39.2
- removed net MISO_PRG: ISP.1, R39.1, U2.(MISO/PCINT3)PB3
- removed net MOSI: IC1.DIN, IC2.A0/NWAIT/MOSI, R37.2, U1.1A
- removed net MOSI_PRG: ISP.4, R37.1, U2.(MOSI/PCINT2)PB2
- removed net N$1: D2.A, IC2.RSTPD, R10.1, R11.2
- removed net N$100: U2.PH1(TXD2), X6.2
- removed net N$12: C54.1, Q7.1, U2.XTAL1
- removed net N$13: C53.1, Q7.2, U2.XTAL2
- removed net N$14: R35.1, X3.DAT1
- removed net N$2: P1.LEDK, Q1.C
- removed net N$3: P1.LEDA@4, R8.1
- removed net N$31: C11.1, IC2.OSCOUT, Q2.1
- removed net N$33: IC2.MFOUT, TP1.TP
- removed net N$34: IC2.VMID, R9.1
- removed net N$35: IC2.AUX, TP2.TP
- removed net N$36: C16.2, C17.1, C20.2, C21.2, L5.2
- removed net N$37: C17.2, R13.2
- removed net N$38: C15.1, C18.1, C19.1, L4.2
- removed net N$39: C18.2, C19.2, C22.1, C24.1, R14.1
- removed net N$4: Q1.B, R2.2
- removed net N$40: R44.1, SP1.+, T3.C
- removed net N$41: R45.2, T3.B
- removed net N$42: PWR.C, R31.1
- removed net N$43: C20.1, C21.1, C23.2, C25.2, R15.1
- removed net N$45: B1.AC1, X7.3
- removed net N$46: B1.AC2, X7.1
- removed net N$47: Q6.D, R38.1
- removed net N$48: D4.C, L8.1, T1.VOUT
- removed net N$49: Q6.S, R36.1
- removed net N$50: Q5.S, R32.1
- removed net N$52: Q5.D, R34.1
- removed net N$53: R33.1, X3.DAT2
- removed net N$54: C10.1, IC2.OSCIN, Q2.2
- removed net N$58: D1.A, P1.RESET, R3.1
- removed net N$6: R47.2, RFID.C
- removed net N$7: P1.LEDA@3, R7.1
- removed net N$8: P1.LEDA@2, R6.1
- removed net N$9: P1.LEDA@1, R5.1
- removed net RX2: U2.PH0(RXD2), X6.1
- removed net RXD: FTDI.2, U2.(RXD0/PCIN8)PE0
- removed net SCK: IC1.DCLK, IC2.A2/SCK, R40.2, U1.2A
- removed net SCK_PRG: ISP.3, R40.1, U2.(SCK/PCINT1)PB1
- removed net SCL: R48.1, U2.(SCL/INT0)PD0, X5.10, X6.4
- removed net SDA: R46.1, U2.(SDA/INT1)PD1, X5.9, X6.3
- removed net TFT_BL: R1.2, R2.1, U2.PL5(OC5C)
- removed net TVDD: C6.1, IC2.TVDD, L1.1
- removed net TXD: FTDI.3, U2.(TXD0)PE1
- removed net VCC: B1.+, C47.+, T1.VIN
- removed net X+: IC1.X+, P1.XR
- removed net X-: IC1.X-, P1.XL
- removed net Y+: IC1.Y+, P1.YD
- removed net Y-: IC1.Y-, P1.YU
- net !RESET_3V3: no longer D1.C, U1.4Y
- net !WIZ_IRQ_3V3: no longer Q5.G, R32.2
- net !WIZ_SS_3V3: no longer U1.6Y
- net +3V3: no longer C1.2, C2.2, C3.2, C50.+, C51.+, C52.1, P1.IM1, P1.IM2, P1.IM3, P1.RD, P1.VCI, P1.VDDI@1, P1.VDDI@2, P1.WRX, PWR.A, R3.2, R33.2, R35.2, T2.OUT, U1.VCC, X3.VDD, X6.6
- net +5V: no longer C13.1, C4.1, C48.+, C49.+, C5.1, C55.1, C56.1, C57.1, C58.1, C59.1, C8.1, C9.1, FTDI.4, IC1.IOVDD, IC1.VCC, IC4.VCC, ISP.2, L1.2, L2.2, L3.2, L8.2, R1.1, R4.2, R41.2, R42.2, R43.2, R44.2, R46.2, R48.2, R49.1, R5.2, R6.2, R7.2, R8.2, RFID.A, SP1.-, T1.FB, T2.IN, U2.AVCC, U2.VCC, U2.VCC1, U2.VCC2, U2.VCC3, X5.8, X6.5
- net GND: no longer B1.-, C1.1, C10.2, C11.2, C12.2, C13.2, C14.2, C15.2, C16.1, C2.1, C22.2, C23.1, C24.2, C25.1, C3.1, C4.2, C47.-, C48.-, C49.-, C5.2, C50.-, C51.-, C52.2, C53.2, C54.2, C55.2, C56.2, C57.2, C58.2, C59.2, C6.2, C60.2, C7.2, C8.2, C9.2, D4.A, FTDI.6, IC1.GND, IC2.A1, IC2.AVSS, IC2.DVSS, IC2.NCS, IC2.TVSS, IC4.VSS, ISP.6, P1.DB0, P1.DB1, P1.DB10, P1.DB11, P1.DB12, P1.DB13, P1.DB14, P1.DB15, P1.DB16, P1.DB17, P1.DB2, P1.DB3, P1.DB4, P1.DB5, P1.DB6, P1.DB7, P1.DB8, P1.DB9, P1.DE, P1.DOTCLK, P1.GND@1, P1.GND@2, P1.GND@3, P1.GND@4, P1.HSYNC, P1.IM0, P1.VSYNC, Q1.E, R11.1, R31.2, T1.!ON!/OFF, T1.GND@3, T1.GND@TAB, T2.GND, T3.E, U1.GND, U2.AGND, U2.GND, U2.GND1, U2.GND2, U2.GND3, X3.GND, X3.GND1, X3.VSS, X5.7, X6.7
- net MISO_3V3: no longer P1.SDO, Q6.G, R36.2, X3.DATA_IN
- net MOSI_3V3: no longer P1.SDI, U1.1Y, X3.DATA_OUT
- net SCK_3V3: no longer P1.D/CX, U1.2Y, X3.SCLK
- net VCC_NET: no longer X7.2
Other:
- note removed: "2.8" Display 320x240"
- note removed: "Antenna-Circuit"
- note removed: "Antenna-Coil"
- note removed: "Buzzer"
- note removed: "Connectors"
- note removed: "Decoupling"
- note removed: "Display"
- note removed: "EMC-Filter"
- note removed: "Level-Shifter"
- note removed: "Low Dropout Regulator (5V -> 3.3V)"
- note removed: "Main-Controller-Unit"
- note removed: "Matching"
- note removed: "Power Jack + Schottky Bridge Rectifier"
- note removed: "Power LED"
- note removed: "Power-Circuit"
- note removed: "RFID-Circuit"
- note removed: "RFID-IC"
- note removed: "RFID_LED"
- note removed: "RX-Circuit"
- note removed: "Reset Circuit"
- note removed: "SD-Card"
- note removed: "Step-Down switching Voltage Regulator (VIN -> 5V)"
- note removed: "Touch Screen Controller"
- note removed: "V1.0"
- note removed: "X8"
